File: CartHeaderBase/CartHeaderBase.kicad_pcb (KiCad board)
At the start: 2 copper layers, 77.3 x 40.1 mm, 9 parts

Commit message: Minor corrections in the comments.
Other:
- board text added: "To ensure it fits on the keyboard socket, use a PCB thickness of 1mm maximum ( 1mm recommended)."
Changed lines of the file:
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@@
   )
   (paper "A4")
+  (title_block
+    (title "Cart header base board")
+    (date "2025-04-04")
+    (rev "0.0")
+    (company "Tolaemon")
+    (comment 1 "http://www.tolaemon.com/dpack/download.htm")
+    (comment 2 "Using this information implies accepting the conditions specified at:")
+  )
   (layers
     (0 "F.Cu" signal)
@@
     (effects (font (size 1.1 1.1) (thickness 0.2)))
   )
+  (gr_text "To ensure it fits on the keyboard socket, use a PCB thickness of 1mm maximum ( 1mm recommended)." (at 156.22 81.11) (layer "Dwgs.User")
+    (effects (font (size 1 1) (thickness 0.15)))
+  )
   (group "" (id 32298dec-8dd6-48a6-91c0-de792069092c)
